File: Electronics/Gyro_Controller.kicad_sch (KiCad schematic)
At the start: 35 parts, among them J3 SWCLK SWD, SW3 SW_Push, SW4 ~{USB_BOOT}, U7 W25Q32JVZP, U8 RP2040, Y2 ABM8-272-T3

Commit message: buttons
Parts:
- C2: footprint (none) -> Capacitor_SMD:C_0805_2012Metric
- R13, R14, R15, R16, R17: footprint (none) -> Resistor_SMD:R_0603_1608Metric
- SW3: value SW_Push -> RST
Changed lines of the file:
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@@
       (effects (font (size 1.27 1.27)))
     )
-    (property "Footprint" "" (at 59.69 154.178 90)
+    (property "Footprint" "Resistor_SMD:R_0603_1608Metric" (at 59.69 154.178 90)
       (effects (font (size 1.27 1.27)) hide)
     )
@@
       (effects (font (size 1.27 1.27)))
     )
-    (property "Footprint" "" (at 31.242 36.83 90)
+    (property "Footprint" "Resistor_SMD:R_0603_1608Metric" (at 31.242 36.83 90)
       (effects (font (size 1.27 1.27)) hide)
     )
@@
       (effects (font (size 1.27 1.27)) (justify left))
     )
-    (property "Footprint" "" (at 199.0852 45.72 0)
+    (property "Footprint" "Capacitor_SMD:C_0805_2012Metric" (at 199.0852 45.72 0)
       (effects (font (size 1.27 1.27)) hide)
     )
@@
       (effects (font (size 1.27 1.27)) (justify right))
     )
-    (property "Value" "SW_Push" (at 21.59 55.88 0)
+    (property "Value" "RST" (at 21.59 55.88 0)
       (effects (font (size 1.27 1.27)) (justify right))
     )
@@
       (effects (font (size 1.27 1.27)))
     )
-    (property "Footprint" "" (at 78.232 163.83 90)
+    (property "Footprint" "Resistor_SMD:R_0603_1608Metric" (at 78.232 163.83 90)
       (effects (font (size 1.27 1.27)) hide)
     )
@@
       (effects (font (size 1.27 1.27)))
     )
-    (property "Footprint" "" (at 55.88 53.848 90)
+    (property "Footprint" "Resistor_SMD:R_0603_1608Metric" (at 55.88 53.848 90)
       (effects (font (size 1.27 1.27)) hide)
     )
@@
       (effects (font (size 1.27 1.27)))
     )
-    (property "Footprint" "" (at 55.88 51.308 90)
-      (effects (font (size 1.27 1.27)) hide)
-    )
+    (property "Footprint" "Resistor_SMD:R_0603_1608Metric" (at 55.88 51.308 90)
+      (effects (font (size 1.27 1.27)) hide)
+    )

Commit message: started pcb, need bigger frame
Parts:
- C2: footprint Capacitor_SMD:C_0805_2012Metric -> Capacitor_SMD:C_0201_0603Metric
- C23, C24, C25, C26, C27, C28, C30, C31, C32, C33, C34, C35, C36, C37, C38, C39, C40, C41, C42: footprint (none) -> Capacitor_SMD:C_0201_0603Metric
- D5: footprint (none) -> LED_SMD:LED_0603_1608Metric
- J3: footprint (none) -> Connector_PinHeader_2.54mm:PinHeader_1x02_P2.54mm_Vertical
- R13, R14, R15, R16, R17: footprint Resistor_SMD:R_0603_1608Metric -> Resistor_SMD:R_0201_0603Metric
- R20: footprint (none) -> Resistor_SMD:R_0201_0603Metric
- SW3: footprint (none) -> Button_Switch_SMD:SW_SPST_TL3342
- SW4: footprint (none) -> Button_Switch_SMD:SW_DPDT_CK_JS202011JCQN
- Y2: footprint (none) -> Crystal:Crystal_SMD_Abracon_ABM8G-4Pin_3.2x2.5mm
Changed lines of the file:
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@@
       (effects (font (size 1.27 1.27)))
     )
-    (property "Footprint" "Resistor_SMD:R_0603_1608Metric" (at 59.69 154.178 90)
+    (property "Footprint" "Resistor_SMD:R_0201_0603Metric" (at 59.69 154.178 90)
       (effects (font (size 1.27 1.27)) hide)
     )
@@
       (effects (font (size 1.27 1.27)) (justify left))
     )
-    (property "Footprint" "" (at 131.7752 31.75 0)
+    (property "Footprint" "Capacitor_SMD:C_0201_0603Metric" (at 131.7752 31.75 0)
       (effects (font (size 1.27 1.27)) hide)
     )
@@
       (effects (font (size 1.27 1.27)))
     )
-    (property "Footprint" "Resistor_SMD:R_0603_1608Metric" (at 31.242 36.83 90)
+    (property "Footprint" "Resistor_SMD:R_0201_0603Metric" (at 31.242 36.83 90)
       (effects (font (size 1.27 1.27)) hide)
     )
@@
       (effects (font (size 1.27 1.27)) (justify left))
     )
-    (property "Footprint" "" (at 267.6652 45.72 0)
+    (property "Footprint" "Capacitor_SMD:C_0201_0603Metric" (at 267.6652 45.72 0)
       (effects (font (size 1.27 1.27)) hide)
     )
@@
       (effects (font (size 1.27 1.27)) (justify left))
     )
-    (property "Footprint" "" (at 124.1552 31.75 0)
+    (property "Footprint" "Capacitor_SMD:C_0201_0603Metric" (at 124.1552 31.75 0)
       (effects (font (size 1.27 1.27)) hide)
     )
@@
       (effects (font (size 1.27 1.27)) (justify left))
     )
-    (property "Footprint" "" (at 229.5652 90.17 0)
+    (property "Footprint" "Capacitor_SMD:C_0201_0603Metric" (at 229.5652 90.17 0)
       (effects (font (size 1.27 1.27)) hide)
     )
@@
       (effects (font (size 1.27 1.27)) (justify left))
     )
-    (property "Footprint" "" (at 237.1852 90.17 0)
+    (property "Footprint" "Capacitor_SMD:C_0201_0603Metric" (at 237.1852 90.17 0)
       (effects (font (size 1.27 1.27)) hide)
     )
@@
       (effects (font (size 1.27 1.27)))
     )
-    (property "Footprint" "" (at 54.61 107.95 0)
+    (property "Footprint" "Connector_PinHeader_2.54mm:PinHeader_1x02_P2.54mm_Vertical" (at 54.61 107.95 0)
       (effects (font (size 1.27 1.27)) hide)
     )
@@
       (effects (font (size 1.27 1.27)))
     )
-    (property "Footprint" "" (at 129.54 95.25 0)
+    (property "Footprint" "LED_SMD:LED_0603_1608Metric" (at 129.54 95.25 0)
       (effects (font (size 1.27 1.27)) hide)
     )
@@
       (effects (font (size 1.27 1.27)) (justify left))
     )
-    (property "Footprint" "Capacitor_SMD:C_0805_2012Metric" (at 199.0852 45.72 0)
+    (property "Footprint" "Capacitor_SMD:C_0201_0603Metric" (at 199.0852 45.72 0)
       (effects (font (size 1.27 1.27)) hide)
     )
@@
       (effects (font (size 1.27 1.27)) (justify left))
     )
-    (property "Footprint" "" (at 33.02 86.6648 0)
+    (property "Footprint" "Capacitor_SMD:C_0201_0603Metric" (at 33.02 86.6648 0)
       (effects (font (size 1.27 1.27)) hide)
     )
@@
       (effects (font (size 1.27 1.27)) (justify left))
     )
-    (property "Footprint" "" (at 244.8052 90.17 0)
+    (property "Footprint" "Capacitor_SMD:C_0201_0603Metric" (at 244.8052 90.17 0)
       (effects (font (size 1.27 1.27)) hide)
     )
@@
       (effects (font (size 1.27 1.27)) (justify left))
     )
-    (property "Footprint" "" (at 207.9752 45.72 0)
+    (property "Footprint" "Capacitor_SMD:C_0201_0603Metric" (at 207.9752 45.72 0)
       (effects (font (size 1.27 1.27)) hide)
     )
@@
       (effects (font (size 1.27 1.27)))
     )
-    (property "Footprint" "" (at 115.57 97.028 90)
+    (property "Footprint" "Resistor_SMD:R_0201_0603Metric" (at 115.57 97.028 90)
       (effects (font (size 1.27 1.27)) hide)
     )
@@
       (effects (font (size 1.27 1.27)) (justify left))
     )
-    (property "Footprint" "" (at 33.02 96.8248 0)
+    (property "Footprint" "Capacitor_SMD:C_0201_0603Metric" (at 33.02 96.8248 0)
       (effects (font (size 1.27 1.27)) hide)
     )
@@
       (effects (font (size 1.27 1.27)) (justify right))
     )
-    (property "Footprint" "" (at 17.78 52.07 0)
+    (property "Footprint" "Button_Switch_SMD:SW_SPST_TL3342" (at 17.78 52.07 0)
       (effects (font (size 1.27 1.27)) hide)
     )
@@
       (effects (font (size 1.27 1.27)))
     )
-    (property "Footprint" "Resistor_SMD:R_0603_1608Metric" (at 78.232 163.83 90)
+    (property "Footprint" "Resistor_SMD:R_0201_0603Metric" (at 78.232 163.83 90)
       (effects (font (size 1.27 1.27)) hide)
     )
@@
       (effects (font (size 1.27 1.27)) (justify left))
     )
-    (property "Footprint" "" (at 33.9852 170.18 0)
+    (property "Footprint" "Capacitor_SMD:C_0201_0603Metric" (at 33.9852 170.18 0)
       (effects (font (size 1.27 1.27)) hide)
     )
@@
       (effects (font (size 1.27 1.27)))
     )
-    (property "Footprint" "Resistor_SMD:R_0603_1608Metric" (at 55.88 53.848 90)
+    (property "Footprint" "Resistor_SMD:R_0201_0603Metric" (at 55.88 53.848 90)
       (effects (font (size 1.27 1.27)) hide)
     )
@@
       (effects (font (size 1.27 1.27)) (justify left))
     )
-    (property "Footprint" "" (at 191.4652 90.17 0)
+    (property "Footprint" "Capacitor_SMD:C_0201_0603Metric" (at 191.4652 90.17 0)
       (effects (font (size 1.27 1.27)) hide)
     )
@@
       (effects (font (size 1.27 1.27)) (justify left))
     )
-    (property "Footprint" "" (at 139.3952 31.75 0)
+    (property "Footprint" "Capacitor_SMD:C_0201_0603Metric" (at 139.3952 31.75 0)
       (effects (font (size 1.27 1.27)) hide)
     )
@@
       (effects (font (size 1.27 1.27)) (justify left))
     )
-    (property "Footprint" "" (at 221.9452 90.17 0)
+    (property "Footprint" "Capacitor_SMD:C_0201_0603Metric" (at 221.9452 90.17 0)
       (effects (font (size 1.27 1.27)) hide)
     )
@@
       (effects (font (size 1.27 1.27)) (justify left))
     )
-    (property "Footprint" "" (at 183.8452 90.17 0)
+    (property "Footprint" "Capacitor_SMD:C_0201_0603Metric" (at 183.8452 90.17 0)
       (effects (font (size 1.27 1.27)) hide)
     )
@@
       (effects (font (size 1.27 1.27)) (justify left))
     )
-    (property "Footprint" "" (at 214.3252 90.17 0)
+    (property "Footprint" "Capacitor_SMD:C_0201_0603Metric" (at 214.3252 90.17 0)
       (effects (font (size 1.27 1.27)) hide)
     )
@@
       (effects (font (size 1.27 1.27)) (justify left))
     )
-    (property "Footprint" "" (at 206.7052 90.17 0)
+    (property "Footprint" "Capacitor_SMD:C_0201_0603Metric" (at 206.7052 90.17 0)
       (effects (font (size 1.27 1.27)) hide)
     )
@@
       (effects (font (size 1.27 1.27)) (justify left))
     )
-    (property "Footprint" "" (at 33.9852 52.07 0)
+    (property "Footprint" "Capacitor_SMD:C_0201_0603Metric" (at 33.9852 52.07 0)
       (effects (font (size 1.27 1.27)) hide)
     )
@@
       (effects (font (size 1.27 1.27)))
     )
-    (property "Footprint" "" (at 41.91 92.71 0)
+    (property "Footprint" "Crystal:Crystal_SMD_Abracon_ABM8G-4Pin_3.2x2.5mm" (at 41.91 92.71 0)
       (effects (font (size 1.27 1.27)) hide)
     )
@@
       (effects (font (size 1.27 1.27)) (justify left))
     )
-    (property "Footprint" "" (at 199.0852 90.17 0)
+    (property "Footprint" "Capacitor_SMD:C_0201_0603Metric" (at 199.0852 90.17 0)
       (effects (font (size 1.27 1.27)) hide)
     )
@@
       (effects (font (size 1.27 1.27)) (justify left))
     )
-    (property "Footprint" "" (at 80.01 173.99 0)
+    (property "Footprint" "Button_Switch_SMD:SW_DPDT_CK_JS202011JCQN" (at 80.01 173.99 0)
       (effects (font (size 1.27 1.27)) hide)
     )
@@
       (effects (font (size 1.27 1.27)) (justify left))
     )
-    (property "Footprint" "" (at 258.7752 45.72 0)
+    (property "Footprint" "Capacitor_SMD:C_0201_0603Metric" (at 258.7752 45.72 0)
       (effects (font (size 1.27 1.27)) hide)
     )
@@
       (effects (font (size 1.27 1.27)))
     )
-    (property "Footprint" "Resistor_SMD:R_0603_1608Metric" (at 55.88 51.308 90)
-      (effects (font (size 1.27 1.27)) hide)
-    )
+    (property "Footprint" "Resistor_SMD:R_0201_0603Metric" (at 55.88 51.308 90)
+      (effects (font (size 1.27 1.27)) hide)
+    )
