File: Electronics/Motor_Controller.kicad_sch (KiCad schematic)
At the start: 43 parts, among them J2 SWCLK SWD, SW1 SW_Push, SW2 ~{USB_BOOT}, U1 RP2040, U4 W25Q32JVZP, Y1 ABM8-272-T3

Commit message: buttons
Parts:
- C1, C10, C11, C12, C13, C14, C15, C3, C4, C5, C6, C7, C8, C9: footprint (none) -> Capacitor_SMD:C_0805_2012Metric
- R10, R11, R12, R2, R3, R4, R5, R6, R7, R8, R9: footprint (none) -> Resistor_SMD:R_0603_1608Metric
Changed lines of the file:
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@@
       (effects (font (size 1.27 1.27)))
     )
-    (property "Footprint" "" (at 52.07 51.308 90)
+    (property "Footprint" "Resistor_SMD:R_0603_1608Metric" (at 52.07 51.308 90)
       (effects (font (size 1.27 1.27)) hide)
     )
@@
       (effects (font (size 1.27 1.27)) (justify left))
     )
-    (property "Footprint" "" (at 191.4652 120.65 0)
+    (property "Footprint" "Capacitor_SMD:C_0805_2012Metric" (at 191.4652 120.65 0)
       (effects (font (size 1.27 1.27)) hide)
     )
@@
       (effects (font (size 1.27 1.27)) (justify left))
     )
-    (property "Footprint" "" (at 183.8452 120.65 0)
+    (property "Footprint" "Capacitor_SMD:C_0805_2012Metric" (at 183.8452 120.65 0)
       (effects (font (size 1.27 1.27)) hide)
     )
@@
       (effects (font (size 1.27 1.27)) (justify left))
     )
-    (property "Footprint" "" (at 160.9852 120.65 0)
+    (property "Footprint" "Capacitor_SMD:C_0805_2012Metric" (at 160.9852 120.65 0)
       (effects (font (size 1.27 1.27)) hide)
     )
@@
       (effects (font (size 1.27 1.27)) (justify left))
     )
-    (property "Footprint" "" (at 228.2952 36.83 0)
+    (property "Footprint" "Capacitor_SMD:C_0805_2012Metric" (at 228.2952 36.83 0)
       (effects (font (size 1.27 1.27)) hide)
     )
@@
       (effects (font (size 1.27 1.27)))
     )
-    (property "Footprint" "" (at 70.612 162.56 90)
+    (property "Footprint" "Resistor_SMD:R_0603_1608Metric" (at 70.612 162.56 90)
       (effects (font (size 1.27 1.27)) hide)
     )
@@
       (effects (font (size 1.27 1.27)) (justify left))
     )
-    (property "Footprint" "" (at 199.0852 120.65 0)
+    (property "Footprint" "Capacitor_SMD:C_0805_2012Metric" (at 199.0852 120.65 0)
       (effects (font (size 1.27 1.27)) hide)
     )
@@
       (effects (font (size 1.27 1.27)) (justify left))
     )
-    (property "Footprint" "" (at 176.2252 120.65 0)
+    (property "Footprint" "Capacitor_SMD:C_0805_2012Metric" (at 176.2252 120.65 0)
       (effects (font (size 1.27 1.27)) hide)
     )
@@
       (effects (font (size 1.27 1.27)))
     )
-    (property "Footprint" "" (at 191.77 34.798 90)
+    (property "Footprint" "Resistor_SMD:R_0603_1608Metric" (at 191.77 34.798 90)
       (effects (font (size 1.27 1.27)) hide)
     )
@@
       (effects (font (size 1.27 1.27)))
     )
-    (property "Footprint" "" (at 259.08 34.798 90)
+    (property "Footprint" "Resistor_SMD:R_0603_1608Metric" (at 259.08 34.798 90)
       (effects (font (size 1.27 1.27)) hide)
     )
@@
       (effects (font (size 1.27 1.27)) (justify left))
     )
-    (property "Footprint" "" (at 206.7052 120.65 0)
+    (property "Footprint" "Capacitor_SMD:C_0805_2012Metric" (at 206.7052 120.65 0)
       (effects (font (size 1.27 1.27)) hide)
     )
@@
       (effects (font (size 1.27 1.27)))
     )
-    (property "Footprint" "" (at 52.07 53.848 90)
+    (property "Footprint" "Resistor_SMD:R_0603_1608Metric" (at 52.07 53.848 90)
       (effects (font (size 1.27 1.27)) hide)
     )
@@
       (effects (font (size 1.27 1.27)) (justify left))
     )
-    (property "Footprint" "" (at 26.3652 168.91 0)
+    (property "Footprint" "Capacitor_SMD:C_0805_2012Metric" (at 26.3652 168.91 0)
       (effects (font (size 1.27 1.27)) hide)
     )
@@
       (effects (font (size 1.27 1.27)))
     )
-    (property "Footprint" "" (at 111.76 53.848 90)
+    (property "Footprint" "Resistor_SMD:R_0603_1608Metric" (at 111.76 53.848 90)
       (effects (font (size 1.27 1.27)) hide)
     )
@@
       (effects (font (size 1.27 1.27)))
     )
-    (property "Footprint" "" (at 271.78 67.31 0)
+    (property "Footprint" "Capacitor_SMD:C_0805_2012Metric" (at 271.78 67.31 0)
       (effects (font (size 1.27 1.27)) hide)
     )
@@
       (effects (font (size 1.27 1.27)) (justify left))
     )
-    (property "Footprint" "" (at 214.3252 120.65 0)
+    (property "Footprint" "Capacitor_SMD:C_0805_2012Metric" (at 214.3252 120.65 0)
       (effects (font (size 1.27 1.27)) hide)
     )
@@
       (effects (font (size 1.27 1.27)) (justify left))
     )
-    (property "Footprint" "" (at 168.6052 120.65 0)
+    (property "Footprint" "Capacitor_SMD:C_0805_2012Metric" (at 168.6052 120.65 0)
       (effects (font (size 1.27 1.27)) hide)
     )
@@
       (effects (font (size 1.27 1.27)))
     )
-    (property "Footprint" "" (at 111.76 97.028 90)
+    (property "Footprint" "Resistor_SMD:R_0603_1608Metric" (at 111.76 97.028 90)
       (effects (font (size 1.27 1.27)) hide)
     )
@@
       (effects (font (size 1.27 1.27)))
     )
-    (property "Footprint" "" (at 111.76 43.688 90)
+    (property "Footprint" "Resistor_SMD:R_0603_1608Metric" (at 111.76 43.688 90)
       (effects (font (size 1.27 1.27)) hide)
     )
@@
       (effects (font (size 1.27 1.27)))
     )
-    (property "Footprint" "" (at 204.47 67.31 0)
+    (property "Footprint" "Capacitor_SMD:C_0805_2012Metric" (at 204.47 67.31 0)
       (effects (font (size 1.27 1.27)) hide)
     )
@@
       (effects (font (size 1.27 1.27)))
     )
-    (property "Footprint" "" (at 52.07 152.908 90)
+    (property "Footprint" "Resistor_SMD:R_0603_1608Metric" (at 52.07 152.908 90)
       (effects (font (size 1.27 1.27)) hide)
     )
@@
       (effects (font (size 1.27 1.27)) (justify left))
     )
-    (property "Footprint" "" (at 160.9852 36.83 0)
+    (property "Footprint" "Capacitor_SMD:C_0805_2012Metric" (at 160.9852 36.83 0)
       (effects (font (size 1.27 1.27)) hide)
     )
@@
       (effects (font (size 1.27 1.27)))
     )
-    (property "Footprint" "" (at 116.84 107.188 90)
+    (property "Footprint" "Resistor_SMD:R_0603_1608Metric" (at 116.84 107.188 90)
       (effects (font (size 1.27 1.27)) hide)
     )
@@
       (effects (font (size 1.27 1.27)))
     )
-    (property "Footprint" "" (at 27.432 36.83 90)
+    (property "Footprint" "Resistor_SMD:R_0603_1608Metric" (at 27.432 36.83 90)
       (effects (font (size 1.27 1.27)) hide)
     )
@@
       (effects (font (size 1.27 1.27)) (justify left))
     )
-    (property "Footprint" "" (at 122.8852 116.84 0)
-      (effects (font (size 1.27 1.27)) hide)
-    )
+    (property "Footprint" "Capacitor_SMD:C_0805_2012Metric" (at 122.8852 116.84 0)
+      (effects (font (size 1.27 1.27)) hide)
+    )

Commit message: started pcb, need bigger frame
Parts:
- C1, C10, C11, C12, C13, C14, C15, C3, C4, C5, C6, C7, C8, C9: footprint Capacitor_SMD:C_0805_2012Metric -> Capacitor_SMD:C_0201_0603Metric
- C16, C17, C18, C19, C20, C21, C22: footprint (none) -> Capacitor_SMD:C_0201_0603Metric
- D2, D3, D4: footprint (none) -> LED_SMD:LED_0603_1608Metric
- J2: footprint (none) -> Connector_PinHeader_2.54mm:PinHeader_1x02_P2.54mm_Vertical
- R10, R11, R12, R2, R3, R4, R5, R6, R7, R8, R9: footprint Resistor_SMD:R_0603_1608Metric -> Resistor_SMD:R_0201_0603Metric
- SW1: footprint (none) -> Button_Switch_SMD:SW_SPST_TL3342
- SW2: footprint (none) -> Button_Switch_SMD:SW_DPDT_CK_JS202011JCQN
- Y1: footprint (none) -> Crystal:Crystal_SMD_Abracon_ABM8G-4Pin_3.2x2.5mm
