File: Electronics/Electronics.kicad_sch (KiCad schematic)
At the start: 20 parts, among them J4 ML, J5 MR, P1 USB_C_Plug_USB2.0, SW5 SW_DIP_x02, U11 AMS1117-3.3, U12 AMS1117-3.3

Commit message: started pcb, need bigger frame
Parts:
- BT1: footprint Battery:BatteryHolder_Keystone_2479_3xAAA -> Battery:BatteryHolder_Keystone_2462_2xAA
- SW5: footprint Button_Switch_SMD:SW_SPST_TL3342 -> Button_Switch_SMD:SW_DIP_SPSTx02_Slide_9.78x7.26mm_W8.61mm_P2.54mm
Changed lines of the file:
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@@
       (effects (font (size 1.27 1.27)) (justify left))
     )
-    (property "Footprint" "Battery:BatteryHolder_Keystone_2479_3xAAA" (at 212.09 125.476 90)
+    (property "Footprint" "Battery:BatteryHolder_Keystone_2462_2xAA" (at 212.09 125.476 90)
       (effects (font (size 1.27 1.27)) hide)
     )
@@
       (effects (font (size 1.27 1.27)))
     )
-    (property "Footprint" "Button_Switch_SMD:SW_SPST_TL3342" (at 158.75 52.07 0)
+    (property "Footprint" "Button_Switch_SMD:SW_DIP_SPSTx02_Slide_9.78x7.26mm_W8.61mm_P2.54mm" (at 158.75 52.07 0)
       (effects (font (size 1.27 1.27)) hide)
     )

Commit message: routing started
Parts:
- removed BT2: 2xAA, Battery:BatteryHolder_Keystone_2462_2xAA, symbol Device:Battery
Connections:
- net VBAT: now also BT1.1 (+)
Other:
- moved on the sheet: BT1, BT3
Changed lines of the file:
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@@
     (stroke (width 0) (type default))
   )
-  (wire (pts (xy 212.09 109.22) (xy 212.09 111.76))
+  (wire (pts (xy 212.09 109.22) (xy 212.09 115.57))
     (stroke (width 0) (type default))
   )
@@
     (stroke (width 0) (type default))
   )
-  (wire (pts (xy 212.09 143.51) (xy 212.09 142.24))
+  (wire (pts (xy 212.09 143.51) (xy 212.09 135.89))
     (stroke (width 0) (type default))
   )
@@
     )
   )
-  (symbol (lib_id "Device:Battery") (at 212.09 127 0) (unit 1)
-    (in_bom yes) (on_board yes) (dnp no) (fields_autoplaced)
-    (property "Reference" "BT1" (at 215.9 125.1585 0)
-      (effects (font (size 1.27 1.27)) (justify left))
-    )
-    (property "Value" "2xAA" (at 215.9 127.6985 0)
-      (effects (font (size 1.27 1.27)) (justify left))
-    )
-    (property "Footprint" "Battery:BatteryHolder_Keystone_2462_2xAA" (at 212.09 125.476 90)
-      (effects (font (size 1.27 1.27)) hide)
-    )
-    (property "Datasheet" "~" (at 212.09 125.476 90)
+  (symbol (lib_id "Device:Battery") (at 212.09 120.65 0) (unit 1)
+    (in_bom yes) (on_board yes) (dnp no) (fields_autoplaced)
+    (property "Reference" "BT1" (at 215.9 118.8085 0)
+      (effects (font (size 1.27 1.27)) (justify left))
+    )
+    (property "Value" "2xAA" (at 215.9 121.3485 0)
+      (effects (font (size 1.27 1.27)) (justify left))
+    )
+    (property "Footprint" "Battery:BatteryHolder_Keystone_2462_2xAA" (at 212.09 119.126 90)
+      (effects (font (size 1.27 1.27)) hide)
+    )
+    (property "Datasheet" "~" (at 212.09 119.126 90)
       (effects (font (size 1.27 1.27)) hide)
     )
@@
     )
   )
-  (symbol (lib_id "Device:Battery") (at 212.09 137.16 0) (unit 1)
-    (in_bom yes) (on_board yes) (dnp no) (fields_autoplaced)
-    (property "Reference" "BT3" (at 215.9 135.3185 0)
-      (effects (font (size 1.27 1.27)) (justify left))
-    )
-    (property "Value" "2xAA" (at 215.9 137.8585 0)
-      (effects (font (size 1.27 1.27)) (justify left))
-    )
-    (property "Footprint" "Battery:BatteryHolder_Keystone_2462_2xAA" (at 212.09 135.636 90)
-      (effects (font (size 1.27 1.27)) hide)
-    )
-    (property "Datasheet" "~" (at 212.09 135.636 90)
+  (symbol (lib_id "Device:Battery") (at 212.09 130.81 0) (unit 1)
+    (in_bom yes) (on_board yes) (dnp no) (fields_autoplaced)
+    (property "Reference" "BT3" (at 215.9 128.9685 0)
+      (effects (font (size 1.27 1.27)) (justify left))
+    )
+    (property "Value" "2xAA" (at 215.9 131.5085 0)
+      (effects (font (size 1.27 1.27)) (justify left))
+    )
+    (property "Footprint" "Battery:BatteryHolder_Keystone_2462_2xAA" (at 212.09 129.286 90)
+      (effects (font (size 1.27 1.27)) hide)
+    )
+    (property "Datasheet" "~" (at 212.09 129.286 90)
       (effects (font (size 1.27 1.27)) hide)
     )
@@
         )
       )
-    )
-  )
-  (symbol (lib_id "Device:Battery") (at 212.09 116.84 0) (unit 1)
-    (in_bom yes) (on_board yes) (dnp no) (fields_autoplaced)
-    (property "Reference" "BT2" (at 215.9 114.9985 0)
-      (effects (font (size 1.27 1.27)) (justify left))
-    )
-    (property "Value" "2xAA" (at 215.9 117.5385 0)
-      (effects (font (size 1.27 1.27)) (justify left))
-    )
-    (property "Footprint" "Battery:BatteryHolder_Keystone_2462_2xAA" (at 212.09 115.316 90)
-      (effects (font (size 1.27 1.27)) hide)
-    )
-    (property "Datasheet" "~" (at 212.09 115.316 90)
-      (effects (font (size 1.27 1.27)) hide)
-    )
-    (pin "2")
-    (pin "1")
-    (instances
-      (project "Electronics"
-        (path "/4c70cac4-2e87-4919-a1c8-fe5f41acf493"
-          (reference "BT2") (unit 1)
-        )
-      )
