File: Electronics/Electronics.kicad_pcb (KiCad board)
At the start: 2 copper layers, 122 x 136 mm, 128 parts, among them J1 Micro_SD_Card_Det_Hirose_DM3AT, J2 SWCLK SWD, J3 SWCLK SWD, J4 ML, J5 MR, P1 USB_C_Plug_USB2.0, SW1 SW_Push, SW10 SW_Push, SW11 SW_Push, SW12 SW_Push, SW13 SW_Push, SW14 SW_Push, SW15 SW_Push, SW2 ~{USB_BOOT}, SW3 RST, SW4 ~{USB_BOOT}, SW5 SW_DIP_x02, SW6 SW_Push, SW7 ~{USB_BOOT}, SW8 SW_Push, SW9 SW_Push, U1 RP2040, U11 AMS1117-3.3, U12 AMS1117-3.3, U4 W25Q32JVZP, U5 ESP32-S3-WROOM-1, U7 W25Q32JVZP, U8 RP2040, Y1 ABM8-272-T3, Y2 ABM8-272-T3

Commit message: started pcb, need bigger frame
Parts:
- added BT1: 2xAA, Battery:BatteryHolder_Keystone_2462_2xAA, F.Cu at (-145.7, -20.3)
- SW1, SW6: value SW_Push -> RST
- SW10, SW11, SW12, SW13, SW14, SW15, SW8, SW9: footprint Button_Switch_SMD:SW_SPST_TL3342 -> Button_Switch_Keyboard:SW_Cherry_MX_1.00u_PCB
- SW5: footprint Button_Switch_SMD:SW_SPST_TL3342 -> Button_Switch_SMD:SW_DIP_SPSTx02_Slide_9.78x7.26mm_W8.61mm_P2.54mm
- moved BT2 290.0 mm to (-179.6, 95.7)
- moved BT3 235.1 mm to (-137.6, 47.4)
- moved SW14 78.9 mm to (-104.0, 22.6)
- moved SW12 59.6 mm to (2.79, 104.4)
- moved SW9 57.8 mm to (-99.1, 116.8)
- moved SW11 57.2 mm to (-104.7, 82.2)
- moved SW15 44.3 mm to (4.11, 82.1)
- moved SW8 41.5 mm to (-97.8, 54.2)
- moved SW10 30.3 mm to (-44.6, 31.3)
- moved SW13 26.6 mm to (-27.2, 37.7)
- moved U13 11.6 mm to (-6.25, 65.1)
- moved U14 11.3 mm to (-1.93, 65.0)
Other:
- board outline removed

Commit message: routing started
Parts:
- removed BT2: 2xAA, Battery:BatteryHolder_Keystone_2462_2xAA
- moved BT1 267.2 mm to (111.3, 52.7), turned to 180 degrees
- moved BT3 260.2 mm to (122.4, 37.7), turned to 0 degrees
- moved U5 217.6 mm to (116.9, 162.6), turned to 180 degrees
- moved C10 192.1 mm to (130.7, 126.9), turned to 90 degrees
- moved C11 190.6 mm to (129.7, 126.9), turned to 90 degrees
- moved C9 189.2 mm to (127.5, 125.2), turned to 90 degrees
- moved SW1 188.8 mm to (140.2, 139.2)
- moved C12 186.5 mm to (126.5, 125.2), turned to 90 degrees
- moved C17 182.5 mm to (125.6, 125.2), turned to 90 degrees
- moved C8 177.5 mm to (111.9, 138.8), turned to 180 degrees
- moved U4 172.0 mm to (111.1, 129.0)
- moved U1 157.4 mm to (117.1, 141.4)
- moved U2 109.9 mm to (-87.5, 182.9)
- moved P1 105.9 mm to (-29.7, 176.3)
- moved SW6 42.2 mm to (-31.6, 93.6)
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Connections:
- BT1 pad 1: Net-(BT1-+) -> /VBAT
Routing:
- net VCC: track 0.00 -> 1.60 mm
Other:
- board outline added: 142 x 156 mm

Commit message: routing started
Parts:
- moved U5 188.9 mm to (136.8, 350.5)
- moved C7 178.4 mm to (114.1, 129.7)
- moved C18 174.2 mm to (115.5, 134.6), turned to 90 degrees
- moved R10 170.0 mm to (118.9, 135.1), turned to -90 degrees
- moved R9 169.9 mm to (118.1, 135.1), turned to -90 degrees
- moved C16 67.4 mm to (-9.34, 134.2)
- moved C10 15.5 mm to (117.2, 134.6)
- moved C9 14.6 mm to (116.3, 134.6)
- moved C11 11.2 mm to (121.5, 134.6)
- moved C12 11.1 mm to (120.7, 134.6)
- moved C17 11.0 mm to (119.8, 134.6)
- moved U4 2.86 mm to (110.0, 131.6)
Routing:
- net /Motor Controller/QSPI_SS: track 0.00 -> 16.2 mm
- net VCC: track 1.60 -> 16.8 mm
- net /Motor Controller/QSPI_SD1: track 0.00 -> 15.0 mm
- net /Motor Controller/QSPI_SD2: track 0.00 -> 13.6 mm
- net /Motor Controller/QSPI_SD3: track 0.00 -> 8.91 mm
- net /Motor Controller/QSPI_SCLK: track 0.00 -> 7.54 mm
- net Net-(U1-VREG_VOUT): track 0.00 -> 7.12 mm
- net /Motor Controller/QSPI_SD0: track 0.00 -> 5.68 mm
- net Net-(U1-USB_DM): track 0.00 -> 2.76 mm
- net Net-(U1-USB_DP): track 0.00 -> 2.57 mm

Commit message: routing esp32 motor controller, need to read up on diff pair
Parts:
- moved BT3 314.7 mm to (-187.5, 92.2)
- moved BT1 298.8 mm to (-187.5, 57.8), turned to 0 degrees
- moved SW1 252.7 mm to (-103.1, 71.1)
- moved C17 235.7 mm to (-104.2, 61.1), turned to 0 degrees
- moved C18 233.6 mm to (-101.8, 48.9), turned to 0 degrees
- moved C7 232.3 mm to (-106.7, 57.6)
- moved R10 231.6 mm to (-99.3, 57.6), turned to 0 degrees
- moved R9 231.4 mm to (-99.3, 55.9), turned to 0 degrees
- moved J1 215.3 mm to (132.5, 170.4), turned to 180 degrees
- moved U10 203.8 mm to (115.5, 167.0), turned to 90 degrees
- moved SW6 202.9 mm to (156.0, 170.9), turned to 90 degrees
- moved R22 202.2 mm to (155.5, 140.5), turned to -90 degrees
- moved R24 200.9 mm to (141.6, 161.8), turned to 90 degrees
- moved U5 200.0 mm to (152.8, 151.1), turned to -90 degrees
- moved R1 198.8 mm to (147.9, 140.4), turned to -90 degrees
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Routing:
- net GND: track 0.00 -> 81.3 mm, vias 0 -> 10
- net /Telemetry and Control Module/SD_CMD: track 0.00 -> 40.1 mm, vias 0 -> 2
- net Net-(U5-EN): track 0.00 -> 34.3 mm, vias 0 -> 2
- net /Telemetry and Control Module/SD_DAT1: track 0.00 -> 33.6 mm
- net /Telemetry and Control Module/SD_DAT0: track 0.00 -> 33.1 mm, vias 0 -> 2
- net /Telemetry and Control Module/SD_DAT2: track 0.00 -> 28.0 mm, vias 0 -> 2
- net /Telemetry and Control Module/SD_DAT3: track 0.00 -> 27.5 mm, vias 0 -> 2
- net /Telemetry and Control Module/SD_CLK: track 0.00 -> 27.2 mm
- net Net-(SW7-A): track 0.00 -> 8.94 mm
- net Net-(U1-VREG_VOUT): track 7.12 -> 0.00 mm
- net VCC: track 16.8 -> 22.4 mm, vias 0 -> 5
- net /D+: track 0.00 -> 3.03 mm
- net /D-: track 0.00 -> 3.01 mm
- net /Motor Controller/QSPI_SD2: track 13.6 -> 16.3 mm
- net Net-(U1-USB_DM): track 2.76 -> 0.00 mm
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Other:
- copper layers 2 -> 4
